File: TrafficSignSchematic/TrafficSign.sch (KiCad schematic (older format))
At the start: 22 parts, among them J1 IDC connector, U1 ATmega328P-PU, U2 SIM800L, Y1 16MHz

Commit message: Full schematic with links to elements
Parts:
- removed L?: 22uH, symbol Device:L
- added CIN2: 680uF, symbol Device:CP
- added COUT2: 330uF, symbol Device:CP
- added D2: 100V/5A, symbol Device:D_Schottky
- added J2: 3.96mm pitch 4-pin polarized connector, Connector_Molex:Molex_KK-396_A-41791-0004_1x04_P3.96mm_Vertical, symbol Connector_Generic:Conn_01x04
- added L2: 33uH, symbol Device:L
- added VR2: LM2596S-5, Package_TO_SOT_SMD:TO-263-5_TabPin3, symbol Regulator_Switching:LM2596S-5
- AE1: footprint (none) -> Connector_Coaxial:SMA_Amphenol_901-144_Vertical
- D1: value 40V/4A -> 100V/5A
- J1: footprint (none) -> Connector_IDC:IDC-Header_2x08_P2.54mm_Vertical
- U2: footprint (none) -> SIM800:Sim800L
- gave numbers to parts that had none: 1
- renumbered CIN to CIN1, COUT to COUT1
Connections:
- net labels removed: IN+, IN-, OUT+, OUT-
- wire segments 137 -> 171
Other:
- note added: "IN+"
- note added: "IN-"
- note added: "OUT+"
- note added: "OUT-"
- moved on the sheet: BT1, CFF, CIN1, COUT1, D1, J1, L1, R1, R2, SC1, U3, VR1
